File: 1800-experiment-1.kicad_pcb (KiCad board)
At the start: 2 copper layers, 232 parts, among them J1 AVR-ISP-6, SW0 KEYSW, SW1 KEYSW, SW10 KEYSW, SW100 KEYSW, SW101 KEYSW, SW102 KEYSW, SW103 KEYSW, SW11 KEYSW, SW12 KEYSW, SW13 KEYSW, SW14 KEYSW, SW15 KEYSW, SW16 KEYSW, SW17 KEYSW, SW18 KEYSW, SW19 KEYSW, SW2 KEYSW, SW20 KEYSW, SW21 KEYSW, SW22 KEYSW, SW23 KEYSW, SW24 KEYSW, SW25 KEYSW, SW26 KEYSW, SW27 KEYSW, SW28 KEYSW, SW29 KEYSW, SW3 KEYSW, SW30 KEYSW, SW31 KEYSW, SW32 KEYSW, SW33 KEYSW, SW34 KEYSW, SW35 KEYSW, SW36 KEYSW, SW37 KEYSW, SW38 KEYSW, SW39 KEYSW, SW4 KEYSW, SW40 KEYSW, SW41 KEYSW, SW42 KEYSW, SW43 KEYSW, SW44 KEYSW, SW45 KEYSW, SW46 KEYSW, SW47 KEYSW, SW48 KEYSW, SW49 KEYSW, SW5 KEYSW, SW50 KEYSW, SW51 KEYSW, SW52 KEYSW, SW53 KEYSW, SW54 KEYSW, SW55 KEYSW, SW56 KEYSW, SW57 KEYSW, SW58 KEYSW, SW59 KEYSW, SW6 KEYSW, SW60 KEYSW, SW61 KEYSW, SW62 KEYSW, SW63 KEYSW, SW64 KEYSW, SW65 KEYSW, SW66 KEYSW, SW67 KEYSW, SW68 KEYSW, SW69 KEYSW, SW7 KEYSW, SW70 KEYSW, SW71 KEYSW, SW72 KEYSW, SW73 KEYSW, SW74 KEYSW, SW75 KEYSW, SW76 KEYSW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

Commit message: pcb design v1
Parts:
- removed the SW102 at (694.9, 197.9)
- removed the SW93 at (606.9, 210.5)
- removed the SW94 at (582.0, 210.5)
- removed the SW95 at (611.7, 190.3)
- added REF**: MountingHole_2.2mm_M2_Pad, cftkb:MountingHole_2.2mm_M2_Pad, F.Cu at (254.6, 180.5)
- added REF**: MountingHole_2.2mm_M2_Pad, cftkb:MountingHole_2.2mm_M2_Pad, F.Cu at (254.6, 154.1)
- added REF**: MountingHole_2.2mm_M2_Pad, cftkb:MountingHole_2.2mm_M2_Pad, F.Cu at (25.4, 180.5)
- added REF**: MountingHole_2.2mm_M2_Pad, cftkb:MountingHole_2.2mm_M2_Pad, F.Cu at (25.4, 154.1)
- added REF**: MountingHole_2.2mm_M2_Pad, cftkb:MountingHole_2.2mm_M2_Pad, F.Cu at (398.3, 154.1)
- added REF**: MountingHole_2.2mm_M2_Pad, cftkb:MountingHole_2.2mm_M2_Pad, F.Cu at (398.3, 180.5)
- SW30: footprint cftkb:SW_Cherry_MX1A_1.00u_PCB-NOSCREEN -> cftkb:SW_Cherry_MX1A_2.00u_PCBNOSCREEN
- SW9, SW93, SW94, SW95: footprint cftkb:SW_Cherry_MX1A_1.00u_PCB-NOSCREEN -> cftkb:SW_Cherry_MX1A_1.25u_PCBNOSCREEN
- moved D33 855.7 mm to (35.6, 163.8), turned to 270 degrees
- moved D77 846.8 mm to (45.1, 160.0), turned to 270 degrees
- moved D64 841.4 mm to (41.9, 167.6), turned to 270 degrees
- moved D79 834.6 mm to (48.3, 161.9), turned to 270 degrees
- moved D0 834.4 mm to (29.2, 160.0), turned to 270 degrees
- moved D34 833.9 mm to (57.7, 167.6), turned to 270 degrees
- moved D49 831.3 mm to (51.3, 163.8), turned to 270 degrees
- moved D65 828.3 mm to (64.0, 161.9), turned to 270 degrees
- moved D16 820.9 mm to (32.4, 161.9), turned to 270 degrees
- moved D19 801.6 mm to (89.5, 167.6), turned to 270 degrees
- moved D66 800.1 mm to (83.2, 163.8), turned to 270 degrees
- moved D35 796.5 mm to (76.8, 160.0), turned to 270 degrees
- moved D50 786.6 mm to (38.7, 165.7), turned to 270 degrees
- moved D17 779.1 mm to (54.5, 165.7), turned to 270 degrees
- moved D68 776.7 mm to (114.9, 163.8), turned to 270 degrees
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Connections:
- SW102 pad 1: (no net) -> col5
- SW102 pad 2: (no net) -> Net-(D83-Pad2)
- SW86 pad 1: (no net) -> col0
- SW86 pad 2: (no net) -> Net-(D77-Pad2)
- SW87 pad 1: (no net) -> col0
- SW87 pad 2: (no net) -> Net-(D77-Pad2)
- SW88 pad 1: (no net) -> col1
- SW88 pad 2: (no net) -> Net-(D79-Pad2)
- SW90 pad 1: (no net) -> col2
- SW90 pad 2: (no net) -> Net-(D81-Pad2)
- SW91 pad 1: (no net) -> col2
- SW91 pad 2: (no net) -> Net-(D81-Pad2)
- SW92 pad 1: (no net) -> col5
- SW92 pad 2: (no net) -> Net-(D83-Pad2)
- SW93 pad 1: (no net) -> col8
- SW93 pad 2: (no net) -> Net-(D51-Pad2)
- SW94 pad 1: (no net) -> col9
- SW94 pad 2: (no net) -> Net-(D78-Pad2)
- SW95 pad 1: (no net) -> col10
- SW95 pad 2: (no net) -> Net-(D82-Pad2)
Routing:
- net col0: track 0.00 -> 445.0 mm
- net col2: track 0.00 -> 429.0 mm
- net col1: track 0.00 -> 417.3 mm
- net col3: track 0.00 -> 353.5 mm
- net col4: track 0.00 -> 347.5 mm
- net col5: track 0.00 -> 344.3 mm
- net col6: track 0.00 -> 309.1 mm
- net col8: track 0.00 -> 304.6 mm
- net col7: track 0.00 -> 275.2 mm
- net col10: track 0.00 -> 268.1 mm
- net col9: track 0.00 -> 261.8 mm
- net col12: track 0.00 -> 239.7 mm
- net col13: track 0.00 -> 237.3 mm
- net col17: track 0.00 -> 219.2 mm, vias 0 -> 1
- net col11: track 0.00 -> 194.9 mm
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- added copper zone on B.Cu, net GND
- added copper zone on F.Cu, net GND
Other:
- board outline added: 384.2 x 172.7 mm

Commit message: refactoring and cleaning up
Parts:
- moved REF** 129.6 mm to (127.6, 154.4)
- moved D100 101.4 mm to (283.2, 160.0)
- moved D98 89.5 mm to (280.0, 167.6)
- moved D76 84.0 mm to (286.4, 161.9)
- moved D99 83.8 mm to (295.9, 167.6)
- moved D94 76.6 mm to (276.9, 165.7)
- moved D12 72.7 mm to (344.2, 177.8)
- moved D97 72.5 mm to (299.1, 160.0)
- moved D87 66.6 mm to (341.0, 177.8)
- moved D93 65.2 mm to (289.6, 163.8)
- moved D84 64.2 mm to (267.3, 160.0)
- moved D48 59.3 mm to (308.6, 165.7)
- moved D13 57.4 mm to (347.3, 177.8)
- moved D92 56.0 mm to (302.3, 161.9)
- moved D88 51.4 mm to (328.3, 177.8)
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Routing:
- net row5: track 0.00 -> 540.6 mm, vias 0 -> 4
- net row4: track 0.00 -> 534.4 mm, vias 0 -> 2
- net row0: track 0.00 -> 521.6 mm, vias 0 -> 2
- net row3: track 0.00 -> 504.4 mm, vias 0 -> 3
- net row2: track 0.00 -> 499.5 mm, vias 0 -> 3
- net row1: track 0.00 -> 493.2 mm, vias 0 -> 4
- net Net-(D76-Pad2): track 0.00 -> 203.8 mm
- net Net-(D99-Pad2): track 0.00 -> 198.2 mm
- net Net-(D97-Pad2): track 0.00 -> 178.5 mm
- net Net-(D93-Pad2): track 0.00 -> 178.4 mm
- net Net-(D92-Pad2): track 0.00 -> 154.2 mm
- net Net-(D48-Pad2): track 0.00 -> 141.1 mm
- net Net-(D89-Pad2): track 0.00 -> 129.4 mm
- net Net-(D32-Pad2): track 0.00 -> 129.3 mm
- net Net-(D31-Pad2): track 0.00 -> 109.8 mm
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Other:
- rule trace_min: 0.2 -> 0

Commit message: inserted m2 standoffs for mounting
Parts:
- added REF**: MountingHole_2.2mm_M2_Pad, cftkb:MountingHole_2.2mm_M2_Pad, F.Cu at (341.6, 302.3)
- added REF**: MountingHole_2.2mm_M2_Pad, cftkb:MountingHole_2.2mm_M2_Pad, F.Cu at (62.2, 283.2)
- added REF**: MountingHole_2.2mm_M2_Pad, cftkb:MountingHole_2.2mm_M2_Pad, F.Cu at (284.5, 283.2)
- added REF**: MountingHole_2.2mm_M2_Pad, cftkb:MountingHole_2.2mm_M2_Pad, F.Cu at (386.1, 207.0)
- added REF**: MountingHole_2.2mm_M2_Pad, cftkb:MountingHole_2.2mm_M2_Pad, F.Cu at (293.4, 207.0)
- added REF**: MountingHole_2.2mm_M2_Pad, cftkb:MountingHole_2.2mm_M2_Pad, F.Cu at (210.8, 207.0)
- added REF**: MountingHole_2.2mm_M2_Pad, cftkb:MountingHole_2.2mm_M2_Pad, F.Cu at (71.1, 207.0)
